File: meishi_ADeL.kicad_pcb (KiCad board)
At the start: 2 copper layers, 91 x 55 mm, 11 parts, among them J1 HRO-TYPE-C-31-M-13B, K11 kailh_pg1350_1u, K12 kailh_pg1350_1u, K13 kailh_pg1350_1u, K14 kailh_pg1350_1u, K15 kailh_pg1350_1u, K21 kailh_pg1350_1u, K22 kailh_pg1350_1u, K23 kailh_pg1350_1u, K24 kailh_pg1350_1u, K25 kailh_pg1350_1u

Commit message: add parts
Parts:
- added REF**: TQFP-32_7x7mm_P0.8mm, Package_QFP:TQFP-32_7x7mm_P0.8mm, B.Cu at (110.0, 23.5)
- added REF**: D_SOD-123, Diode_SMD:D_SOD-123, B.Cu at (74.9, 29.0)
- added REF**: D_SOD-123, Diode_SMD:D_SOD-123, B.Cu at (74.9, 25.1)
- added REF**1: D_SOD-123, Diode_SMD:D_SOD-123, B.Cu at (78.7, 29.0)
- added REF**2: D_SOD-123, Diode_SMD:D_SOD-123, B.Cu at (78.7, 25.1)
- added REF**3: D_SOD-123, Diode_SMD:D_SOD-123, B.Cu at (82.5, 29.0)
- added REF**4: D_SOD-123, Diode_SMD:D_SOD-123, B.Cu at (82.5, 25.1)
- added REF**5: D_SOD-123, Diode_SMD:D_SOD-123, B.Cu at (86.4, 29.0)
- added REF**6: D_SOD-123, Diode_SMD:D_SOD-123, B.Cu at (86.4, 25.1)
- added REF**7: D_SOD-123, Diode_SMD:D_SOD-123, B.Cu at (90.2, 29.0)
- added REF**8: D_SOD-123, Diode_SMD:D_SOD-123, B.Cu at (90.2, 25.1)
Routing:
- net Row0: track 0.00 -> 15.2 mm
- net Row1: track 0.00 -> 15.2 mm
- net Col3: track 0.00 -> 10.6 mm, vias 0 -> 2
- net Col4: track 0.00 -> 10.6 mm, vias 0 -> 2
- net Col2: track 0.00 -> 10.6 mm, vias 0 -> 2
- net Col1: track 0.00 -> 10.6 mm, vias 0 -> 2
- net Col0: track 0.00 -> 10.6 mm, vias 0 -> 2
Other:
- board text added: "{ name: [{dblquote}Teppei Yoshikawa{dblquote}, {dblquote}ADeL{dblquote}, {dblquote}EwdErna{dblquote}], job: [{ MEITEC: Engineer }], interest: [{dblquote}Development{dblquote}, {dblquote}Keyboard{dblquote}, {dblquote}Music{dblquote}] }"
